File: AVRDevBoardRev1.1.kicad_pcb (KiCad board)
At the start: 2 copper layers, 68 x 53 mm, 35 parts, among them J1 externalPower, J2 Power, J3 PTiny/PD, J4 PB/PC, J5 Barrel_Jack_Switch, J6 ICSP, J7 ICSP, SW1 powerSwitch, SW2 resetButton, U1 AMS1117-5.0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

Commit message: Added dog logo, added microcontroller silkscreen labels, shipped to jlcpcb
Parts:
- added G***: LOGO, graphics:dog2, F.Cu at (116.3, 133.3)
Routing:
- net GND: track 75.3 -> 69.3 mm
Other:
- board text added: "ATMEGA8/ATMEGA328"
- board text added: "ATTINY85"
